File: elec/PCB USB/PCB USB.kicad_pcb (KiCad board)
At the start: 2 copper layers, 0 parts

Commit message: push sélection pièces et schéma électrique clean up
Parts:
- added C201: 0.1uF, Capacitor_SMD:C_0603_1608Metric, F.Cu at (54.2, 47.8)
- added C202: 0.1uF, Capacitor_SMD:C_0603_1608Metric, F.Cu at (54.2, 50.3)
- added C203: 0.1uF, Capacitor_SMD:C_0603_1608Metric, F.Cu at (54.2, 52.8)
- added C204: 0.1uF, Capacitor_SMD:C_0603_1608Metric, F.Cu at (54.2, 55.3)
- added C205: 0.1uF, Capacitor_SMD:C_0603_1608Metric, F.Cu at (54.2, 57.9)
- added C206: 0.1uF, Capacitor_SMD:C_0603_1608Metric, F.Cu at (54.2, 60.4)
- added C207: 0.1uF, Capacitor_SMD:C_0603_1608Metric, F.Cu at (58.2, 47.8)
- added C208: 0.1uF, Capacitor_SMD:C_0603_1608Metric, F.Cu at (58.2, 50.3)
- added C209: 4.7uF, Capacitor_SMD:C_0603_1608Metric, F.Cu at (58.2, 52.8)
- added C210: 0.1uF, Capacitor_SMD:C_0603_1608Metric, F.Cu at (58.2, 55.3)
- added C211: 0.1uF, Capacitor_SMD:C_0603_1608Metric, F.Cu at (58.2, 57.9)
- added C212: 0.1uF, Capacitor_SMD:C_0603_1608Metric, F.Cu at (58.2, 60.4)
- added C213: 10uF, Capacitor_SMD:C_0603_1608Metric, F.Cu at (62.2, 47.8)
- added C214: 12pF, Capacitor_SMD:C_0603_1608Metric, F.Cu at (62.2, 50.3)
- added C215: 12pF, Capacitor_SMD:C_0603_1608Metric, F.Cu at (62.2, 52.8)
- added C216: 4.7uF, Capacitor_SMD:C_0603_1608Metric, F.Cu at (62.2, 55.3)
- added C217: 0.1uF, Capacitor_SMD:C_0603_1608Metric, F.Cu at (62.2, 57.9)
- added C218: 1uF, Capacitor_SMD:C_0603_1608Metric, F.Cu at (62.2, 60.4)
- added C301: 10µF, Capacitor_SMD:C_0805_2012Metric_Pad1.18x1.45mm_HandSolder, F.Cu at (30.1, 65.5)
- added C302: 4,7µF, Capacitor_SMD:C_0805_2012Metric_Pad1.18x1.45mm_HandSolder, F.Cu at (30.1, 68.5)
- added C303: 0.1µF, Capacitor_SMD:C_0603_1608Metric_Pad1.08x0.95mm_HandSolder, F.Cu at (15.7, 55.1)
- added C304: 4,7µF, Capacitor_SMD:C_0805_2012Metric_Pad1.18x1.45mm_HandSolder, F.Cu at (30.1, 71.5)
- added C305: 33pF, Capacitor_SMD:C_0603_1608Metric_Pad1.08x0.95mm_HandSolder, F.Cu at (15.7, 57.6)
- added C306: 22µF, Capacitor_SMD:C_0805_2012Metric_Pad1.18x1.45mm_HandSolder, F.Cu at (30.1, 74.5)
- added C307: 0.1µF, Capacitor_SMD:C_0603_1608Metric_Pad1.08x0.95mm_HandSolder, F.Cu at (15.7, 60.1)
- added C401: 10µF, Capacitor_SMD:C_0603_1608Metric, F.Cu at (34.2, 36.4)
- added C402: 10µF, Capacitor_SMD:C_0603_1608Metric, F.Cu at (34.2, 38.9)
- added C403: 1µF, Capacitor_SMD:C_0603_1608Metric, F.Cu at (34.2, 41.4)
- added C501: 1n, Capacitor_SMD:C_0603_1608Metric, F.Cu at (75.7, 16.2)
- added C502: 1n, Capacitor_SMD:C_0603_1608Metric, F.Cu at (75.7, 18.7)
- added C503: 100n, Capacitor_SMD:C_0603_1608Metric, F.Cu at (75.7, 21.2)
- added D301: Green_power, Diode_SMD:D_0805_2012Metric, F.Cu at (20.1, 73.8)
- added D401: PORT1, Diode_SMD:D_0805_2012Metric, F.Cu at (42.5, 36.6)
- added D402: PORT2, Diode_SMD:D_0805_2012Metric, F.Cu at (42.5, 39.7)
- added D403: PORT3, Diode_SMD:D_0805_2012Metric, F.Cu at (42.5, 42.7)
- added D404: PORT4, Diode_SMD:D_0805_2012Metric, F.Cu at (42.5, 45.8)
- added D405: ACTIVE, Diode_SMD:D_0805_2012Metric, F.Cu at (42.5, 48.8)
- added F301: SMD0805B110TF, Fuse:Fuse_0805_2012Metric, F.Cu at (24.5, 73.8)
- added F401: SMD0805B110TF, Fuse:Fuse_0805_2012Metric, F.Cu at (28.0, 49.6)
- added FB301: 600 @ 100MHz, Resistor_SMD:R_0805_2012Metric_Pad1.20x1.40mm_HandSolder, F.Cu at (30.4, 60.0)
- added FB401: 600 @ 100MHz, Resistor_SMD:R_0805_2012Metric_Pad1.20x1.40mm_HandSolder, F.Cu at (47.1, 50.3)
- added H401: MountingHole, MountingHole:MountingHole_2.2mm_M2, F.Cu at (46.9, 17.9)
- added H402: MountingHole, MountingHole:MountingHole_2.2mm_M2, F.Cu at (46.9, 23.9)
- added J201: USB_C_PICO, Connector_USB:USB_C_Receptacle_G-Switch_GT-USB-7010ASV, F.Cu at (58.1, 67.0)
- added J402: USB_C_Receptacle_USB2.0_14P, Connector_USB:USB_C_Receptacle_G-Switch_GT-USB-7010ASV, F.Cu at (38.1, 20.3)
- added J403: USB_A, Connector_USB:USB_A_CONNFLY_DS1095-WNR0, F.Cu at (19.4, 17.5)
- added J404: USB_C_Receptacle_USB2.0_14P, Connector_USB:USB_C_Receptacle_G-Switch_GT-USB-7010ASV, F.Cu at (38.1, 30.4)
- added J405: USB_A, Connector_USB:USB_A_CONNFLY_DS1095-WNR0, F.Cu at (19.4, 34.1)
- added J501: Conn_I2C_Écran, Connector_PinSocket_2.54mm:PinSocket_1x04_P2.54mm_Vertical, F.Cu at (54.5, 34.6)
- added L201: 3.3uH, Resistor_SMD:R_0805_2012Metric, F.Cu at (54.4, 73.2)
- added L301: 2.2uH 13.2mOhm, Inductor_SMD:L_TDK_VLP8040, F.Cu at (23.0, 58.9)
- added Q301: AO3401A, Package_TO_SOT_SMD:SOT-23, F.Cu at (30.5, 56.3)
- added Q401: AO3401A, Package_TO_SOT_SMD:SOT-23, F.Cu at (47.1, 46.6)
- added R201: 5.1k, Resistor_SMD:R_0603_1608Metric_Pad0.98x0.95mm_HandSolder, F.Cu at (77.1, 69.5)
- added R202: 5.1k, Resistor_SMD:R_0603_1608Metric_Pad0.98x0.95mm_HandSolder, F.Cu at (77.1, 72.0)
- added R203: 100K, Resistor_SMD:R_0603_1608Metric, F.Cu at (66.3, 47.8)
- added R204: 2K, Resistor_SMD:R_0603_1608Metric, F.Cu at (66.3, 50.3)
- added R205: 27, Resistor_SMD:R_0603_1608Metric, F.Cu at (66.3, 52.8)
- added R206: 27, Resistor_SMD:R_0603_1608Metric, F.Cu at (66.3, 55.3)
- added R207: 27, Resistor_SMD:R_0603_1608Metric, F.Cu at (66.3, 57.9)
- added R208: 100K, Resistor_SMD:R_0603_1608Metric, F.Cu at (66.3, 60.4)
- added R301: 100k, Resistor_SMD:R_0603_1608Metric_Pad0.98x0.95mm_HandSolder, F.Cu at (15.7, 62.6)
- added R302: 17.4k, Resistor_SMD:R_0603_1608Metric_Pad0.98x0.95mm_HandSolder, F.Cu at (15.7, 65.2)
- added R303: 330, Resistor_SMD:R_0603_1608Metric_Pad0.98x0.95mm_HandSolder, F.Cu at (15.7, 67.7)
- added R304: 220k, Resistor_SMD:R_0603_1608Metric_Pad0.98x0.95mm_HandSolder, F.Cu at (15.7, 70.2)
- added R305: 30k, Resistor_SMD:R_0603_1608Metric_Pad0.98x0.95mm_HandSolder, F.Cu at (15.7, 72.7)
- added R401: 5.1k, Resistor_SMD:R_0603_1608Metric_Pad0.98x0.95mm_HandSolder, F.Cu at (34.4, 48.9)
- added R403: 5.1k, Resistor_SMD:R_0603_1608Metric, F.Cu at (34.2, 43.9)
- added R404: 5.1k, Resistor_SMD:R_0603_1608Metric, F.Cu at (34.2, 46.4)
- added R405: 220, Resistor_SMD:R_0603_1608Metric, F.Cu at (38.2, 36.4)
- added R406: 220, Resistor_SMD:R_0603_1608Metric, F.Cu at (38.2, 38.9)
- added R407: 470, Resistor_SMD:R_0603_1608Metric, F.Cu at (38.2, 41.4)
- added R408: 5.1k, Resistor_SMD:R_0603_1608Metric, F.Cu at (38.2, 43.9)
- added R409: 5.1k, Resistor_SMD:R_0603_1608Metric, F.Cu at (38.2, 46.4)
- added R501: 10k, Resistor_SMD:R_0603_1608Metric, F.Cu at (75.7, 23.7)
- added R502: 10k, Resistor_SMD:R_0603_1608Metric, F.Cu at (75.7, 26.2)
- added R503: 10k, Resistor_SMD:R_0603_1608Metric, F.Cu at (75.7, 28.8)
- added SW201: SW_BOOTSEL, Button_Switch_SMD:SW_SPST_B3U-1000P, F.Cu at (66.8, 63.8)
- added SW202: SW_RESET, Button_Switch_SMD:SW_SPST_B3U-1000P, F.Cu at (66.8, 68.1)
- added SW501: RotaryEncoder_Switch, Rotary_Encoder:RotaryEncoder_Bourns_Horizontal_PEC12R-2x17F-Sxxxx, F.Cu at (67.0, 21.1)
- added TP301: TP_VIN_5V, TestPoint:TestPoint_Pad_D1.0mm, F.Cu at (34.1, 65.5)
- added TP302: TP_3v3, TestPoint:TestPoint_Pad_D1.0mm, F.Cu at (34.1, 68.6)
- added TP303: TP_5V, TestPoint:TestPoint_Pad_D1.0mm, F.Cu at (34.1, 71.6)
- added TP304: TP_GND, TestPoint:TestPoint_Pad_1.0x1.0mm, F.Cu at (34.1, 74.7)
- added U201: SRV05-4, Package_TO_SOT_SMD:SOT-23-6, F.Cu at (72.3, 70.6)
- added U202: RP2350B-QFN80, Package_DFN_QFN:QFN-80-1EP_10x10mm_P0.4mm_EP3.4x3.4mm_ThermalVias, F.Cu at (74.4, 52.7)
- added U203: W25Q128JVPIQ, Package_SON:WSON-8-1EP_6x5mm_P1.27mm_EP3.4x4mm, F.Cu at (74.0, 65.0)
- added U301: AP7361C-33E, Package_TO_SOT_SMD:SOT-223-3_TabPin2, F.Cu at (22.8, 68.2)
- added U302: ~, Package_TO_SOT_SMD:SOT-563, F.Cu at (15.7, 75.4)
- added U401: SRV05-4, Package_TO_SOT_SMD:SOT-23-6, F.Cu at (47.3, 37.5)
- added U402: ~, Package_DFN_QFN:HVQFN-24-1EP_4x4mm_P0.5mm_EP2.6x2.6mm, F.Cu at (47.1, 30.0)
- added Y201: CM4012M00012001, Crystal:Crystal_SMD_2520-4Pin_2.5x2.0mm, F.Cu at (66.1, 72.3)
- added Y401: 12MHz, Crystal:Crystal_SMD_3225-4Pin_3.2x2.5mm, F.Cu at (47.3, 42.0)
Other:
- board outline added: 75 x 25 mm
- board text added: ": Inside Laptop"
- board text added: ": Outside Laptop"
- board text added: "Note : peut être plus petit, c'est pas mal le plus gros qu'on peut aller ex: le `21` peut être plus proche du 10 afin de laisser juste assez de place pour le conn"
