File: elec/PCB USB/PCB USB.kicad_pcb (KiCad board)
At the start: 4 copper layers, 91 x 38 mm, 88 parts, among them J402 USB_C_Receptacle_USB2.0_14P, J403 USB_A, J404 USB_C_Receptacle_USB2.0_14P, J405 USB_A, P1 USB_C_Plug_USB2.0, Q301 AO3401A, Q401 AO3401A, SW501 RotaryEncoder_Switch, U201 SRV05-4, U202 RP2350B-QFN80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

Commit message: push crystal fix
Connections:
- Y401 pad 2: (no net) -> GND
- Y401 pad 4: (no net) -> GND
Routing:
- net GND: track 57.3 -> 60.4 mm

Commit message: push kicad fix
Parts:
- removed 5V: TP_VIN_5V, TestPoint:TestPoint_Pad_D1.0mm
- removed BOOT: SW_BOOTSEL, Button_Switch_SMD:SW_SPST_B3U-1000P
- removed PICO: USB_C_PICO, Connector_USB:USB_C_Receptacle_G-Switch_GT-USB-7010ASV
- removed REF**: OSHW-Symbol_13.4x12mm_SilkScreen, Symbol:OSHW-Symbol_13.4x12mm_SilkScreen
- removed REF**: KiCad-Logo_8mm_SilkScreen, Symbol:KiCad-Logo_8mm_SilkScreen
- removed RST: SW_RESET, Button_Switch_SMD:SW_SPST_B3U-1000P
- removed U201: SRV05-4, Package_TO_SOT_SMD:SOT-23-6
- added 5v: TP_VIN_5V, TestPoint:TestPoint_Pad_D1.0mm, F.Cu at (91.5, 115.3)
- added DEBUG: DEBUG, Connector_PinHeader_1.27mm:PinHeader_1x03_P1.27mm_Vertical, F.Cu at (140.4, 107.5)
- added J201: USB_C_PICO, Connector_USB:USB_C_Receptacle_G-Switch_GT-USB-7010ASV, F.Cu at (86.9, 84.4)
- added R209: 1k, Resistor_SMD:R_0603_1608Metric, F.Cu at (150.7, 106.5)
- added SW201: SW_BOOTSEL, Button_Switch_SMD:SW_SPST_B3U-1000P, F.Cu at (87.5, 114.5)
- added SW202: SW_RESET, Button_Switch_SMD:SW_SPST_B3U-1000P, F.Cu at (87.5, 110.5)
- R203: value 100K -> 10k
- R204: value 2K -> 1k
- R208: value 100K -> NP
- moved C214 0.43 mm to (146.3, 108.7)
- moved C215 0.43 mm to (151.5, 108.7)
- moved Y201 0.43 mm to (148.9, 108.7)
Connections:
- C215 pad 1: Net-(U202-XOUT) -> Net-(C215-Pad1)
- R206 pad 1: /MCU/D- -> /MCU/D+
- R206 pad 2: /MCU/USB_PICO_D- -> /MCU/USB_PICO_D+
- R207 pad 1: /MCU/USB_PICO_D+ -> /MCU/USB_PICO_D-
- R207 pad 2: /MCU/D+ -> /MCU/D-
- U202 pad 66: /MCU/D+ -> /MCU/D-
- U202 pad 67: /MCU/D- -> /MCU/D+
- Y201 pad 1: Net-(U202-XOUT) -> Net-(C215-Pad1)
Routing:
- net /MCU/USB_PICO_D+: track 36.4 -> 9.63 mm
- net /MCU/USB_PICO_D-: track 34.1 -> 10.4 mm
- net /MCU/SWCLK: track 0.00 -> 17.5 mm, vias 0 -> 1
- net /MCU/SWDIO: track 0.00 -> 16.8 mm, vias 0 -> 1
- net GND: track 60.4 -> 65.8 mm, vias 112 -> 87
- net Net-(C215-Pad1): track 0.00 -> 3.24 mm
- net +5V: track 117.8 -> 114.7 mm
- net Net-(U202-XOUT): track 4.56 -> 1.72 mm
- net /MCU/D+: track 62.4 -> 64.7 mm
- net +3V3: track 178.9 -> 181.1 mm
- net VBUS: track 252.0 -> 250.3 mm
- net Net-(U202-XIN): track 8.98 -> 7.41 mm, vias 2 -> 0
