File: elec/PCB USB/MCU.kicad_sch (KiCad schematic)
At the start: 34 parts, among them J1 USB_C_PICO, SW1 SW_BOOTSEL, SW2 SW_RESET, U1 SRV05-4, U2 RP2350B-QFN80, U3 W25Q128JVPIQ, Y1 CM4012M00012001

Commit message: push sélection pièces et schéma électrique clean up
Parts:
- renumbered C1 to C201, C2 to C202, C3 to C203, C4 to C204, C5 to C205, C6 to C206, C7 to C207, C8 to C208, C9 to C209, C10 to C210, C11 to C211, C12 to C212, C13 to C213, C14 to C214, C15 to C215, C16 to C216, C17 to C217, C18 to C218, J1 to J201, L1 to L201, R1 to R201, R2 to R202, R3 to R203, R4 to R204, R5 to R205, R6 to R206, R7 to R207, R8 to R208, SW1 to SW201, SW2 to SW202, U1 to U201, U2 to U202, U3 to U203, Y1 to Y201
Connections:
- net VBUS_USB_5V renamed VBUS
Other:
- note added: "Encodeur"
- note removed: "M_Conn_LEFT"
- note removed: "M_Conn_RIGHT"

Commit message: push pcb
Parts:
- C209, C213, C216: footprint Capacitor_SMD:C_0603_1608Metric -> Capacitor_SMD:C_0805_2012Metric
Changed lines of the file:
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@@
 			)
 		)
-		(property "Footprint" "Capacitor_SMD:C_0603_1608Metric"
+		(property "Footprint" "Capacitor_SMD:C_0805_2012Metric"
 			(at 212.09 48.26 0)
 			(effects
@@
 			)
 		)
-		(property "Footprint" "Capacitor_SMD:C_0603_1608Metric"
+		(property "Footprint" "Capacitor_SMD:C_0805_2012Metric"
 			(at 146.05 59.69 0)
 			(effects
@@
 			)
 		)
-		(property "Footprint" "Capacitor_SMD:C_0603_1608Metric"
+		(property "Footprint" "Capacitor_SMD:C_0805_2012Metric"
 			(at 146.05 86.36 0)
 			(effects

Commit message: push kicad fix
Parts:
- removed U201: SRV05-4, Package_TO_SOT_SMD:SOT-23-6, symbol Power_Protection:SRV05-4
- added J202: DEBUG, Connector_PinHeader_2.54mm:PinHeader_1x03_P2.54mm_Vertical, symbol Connector:Conn_01x03_Socket
- added R209: 1k, Resistor_SMD:R_0603_1608Metric, symbol Device:R_US
- R203: value 100K -> 10k
- R204: value 2K -> 1k
- R208: value 100K -> NP
Connections:
- net D+: now also R206.1, U202.67 (USB_DP); no longer R207.2, U202.66 (USB_DM)
- net D-: now also R207.2, U202.66 (USB_DM); no longer R206.1, U202.67 (USB_DP)
- net GND: now also J202.2 (Pin_2)
- net SWCLK: now also J202.1 (Pin_1)
- net SWDIO: now also J202.3 (Pin_3)
- net USB_PICO_D+: now also R206.2; no longer R207.1
- net USB_PICO_D-: now also R207.1; no longer R206.2
- net at C215.1, Y201.1: now also R209.1; no longer U202.31 (XOUT)
- new net: R209.2, U202.31 (XOUT)
Other:
- moved on the sheet: C214, C215, R203, SW202, Y201

Commit message: Push non terminé
Other:
- company: (none) -> C3I
- title: (none) -> Hub USB2.0 Pomodoro
Changed lines of the file:
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@@
 	(generator "eeschema")
 	(generator_version "9.0")
-	(paper "B")
+	(paper "A3")
+	(title_block
+		(title "Hub USB2.0 Pomodoro")
+		(date "2025-04-20")
+		(rev "1.0")
+		(company "C3I")
+		(comment 1 "Jacob Turcotte")
+		(comment 2 "&")
+		(comment 3 "Charles-Ariel Dion")
+		(comment 4 "Par: Équipe 3")
+	)
 	(text "Encodeur"
 		(exclude_from_sim no)
