File: elec/PCB USB/USB_HUB.kicad_sch (KiCad schematic)
At the start: 13 parts, among them P1 USB_C_Plug_USB2.0, Q2 AO3401A, U5 SRV05-4, Y2 12MHz

Commit message: push schema
Parts:
- added J3, J5: USB_A, symbol Connector:USB_A
- added J4, J6: USB_C_Receptacle_USB2.0_14P, symbol Connector:USB_C_Receptacle_USB2.0_14P
- added R18, R19, R20, R21: 5.1k, symbol Device:R_US
Connections:
- net GND: now also J3.4 (GND), J3.5 (Shield), J4.A1 (GND), J4.A12 (GND), J4.B1 (GND), J4.B12 (GND), J4.S1 (SHIELD), J5.4 (GND), J5.5 (Shield), J6.A1 (GND), J6.A12 (GND), J6.B1 (GND), J6.B12 (GND), J6.S1 (SHIELD), R18.2, R19.2, R20.2, R21.2
- net USBA_2_D+: now reaches U7.10 (D_{+2})
- net USBA_2_D+: now also J5.2 (D-)
- net USBC_1_D-: now reaches U7.11 (D_{-1})
- net USBC_1_D-: now also J4.A7 (D-), J4.B7 (D-)
- net USBC_1_D+: now reaches U7.12 (D_{+1})
- net USBC_1_D+: now also J4.A6 (D+), J4.B6 (D+)
- net USBC_2_D-: now reaches U7.5 (D_{-4})
- net USBC_2_D-: now also J6.A7 (D-), J6.B7 (D-)
- net USBC_2_D+: now reaches U7.6 (D_{+4})
- net USBC_2_D+: now also J6.A6 (D+), J6.B6 (D+)
- net USBA_1_D-: now reaches U7.7 (D_{-3})
- net USBA_1_D-: now also J3.3 (D+)
- net USBA_1_D+: now reaches U7.8 (D_{+3})
- net USBA_1_D+: now also J3.2 (D-)
- net USBA_2_D-: now reaches U7.9 (D_{-2})
- net USBA_2_D-: now also J5.3 (D+)
- new net: J4.B5 (CC2), R19.1
- new net: J6.A5 (CC1), R20.1
- new net: J6.B5 (CC2), R21.1
- new net: J4.A5 (CC1), R18.1
- new net VCC: J3.1 (VBUS), J4.A4 (VBUS), J4.A9 (VBUS), J4.B4 (VBUS), J4.B9 (VBUS), J5.1 (VBUS), J6.A4 (VBUS), J6.A9 (VBUS), J6.B4 (VBUS), J6.B9 (VBUS)
Other:
- moved on the sheet: C23, C27, C28, U7, Y2

Commit message: push sélection pièces et schéma électrique clean up
Parts:
- removed R14: 5.1k, Resistor_SMD:R_0603_1608Metric, symbol Device:R_US
- added D401: PORT1, Diode_SMD:D_0805_2012Metric, symbol Device:LED
- added D402: PORT2, Diode_SMD:D_0805_2012Metric, symbol Device:LED
- added D403: PORT3, Diode_SMD:D_0805_2012Metric, symbol Device:LED
- added D404: PORT4, Diode_SMD:D_0805_2012Metric, symbol Device:LED
- added D405: ACTIVE, Diode_SMD:D_0805_2012Metric, symbol Device:LED
- added R401: 5.1k, Resistor_SMD:R_0603_1608Metric_Pad0.98x0.95mm_HandSolder, symbol Device:R_US
- added R405, R406: 220, Resistor_SMD:R_0603_1608Metric, symbol Device:R_US
- added R407: 470, Resistor_SMD:R_0603_1608Metric, symbol Device:R_US
- J402: renamed from J6; footprint (none) -> Connector_USB:USB_C_Receptacle_G-Switch_GT-USB-7010ASV
- J403: renamed from J5; footprint (none) -> Connector_USB:USB_A_CONNFLY_DS1095-WNR0
- J404: renamed from J4; footprint (none) -> Connector_USB:USB_C_Receptacle_G-Switch_GT-USB-7010ASV
- J405: renamed from J3; footprint (none) -> Connector_USB:USB_A_CONNFLY_DS1095-WNR0
- R403: renamed from R20; footprint (none) -> Resistor_SMD:R_0603_1608Metric
- R404: renamed from R21; footprint (none) -> Resistor_SMD:R_0603_1608Metric
- R408: renamed from R18; footprint (none) -> Resistor_SMD:R_0603_1608Metric
- R409: renamed from R19; footprint (none) -> Resistor_SMD:R_0603_1608Metric
- renumbered C23 to C401, C27 to C402, C28 to C403, F2 to F401, FB2 to FB401, H1 to H401, H2 to H402, Q2 to Q401, U5 to U401, U7 to U402, Y2 to Y401
Connections:
- net VCC is gone; now on net VBUS: J402.A4 (VBUS), J402.A9 (VBUS), J402.B4 (VBUS), J402.B9 (VBUS), J403.1 (VBUS), J404.A4 (VBUS), J404.A9 (VBUS), J404.B4 (VBUS), J404.B9 (VBUS), J405.1 (VBUS)
- net +3V3: now also D405.2 (A)
- net GND: now also R401.2
- net at P1.A5 (CC): now also R401.1
- net at U402.21 (LED_{4}/SDA): now also D401.2 (A), D402.1 (K), D403.2 (A), D404.1 (K), R407.2
- net at U402.22 (LED_{1}): now also R405.2
- net at U402.23 (LED_{2}): now also R406.2
- new net: D401.1 (K), D402.2 (A), R405.1
- new net: D403.1 (K), D404.2 (A), R406.1
- no-connect marks 5 -> 6
Other:
- moved on the sheet: J403, J405, P1

Commit message: PUSHHHHHHHHHHHH
Parts:
- P1: footprint JT_USB_C_PLUG2-0:UP20-C-F-G-FL-1-P12-TR -> JT_USB_C:UP20-C-F-G-FL-1-P12-TR
Changed lines of the file:
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@@
 			)
 		)
-		(property "Footprint" "JT_USB_C_PLUG2-0:UP20-C-F-G-FL-1-P12-TR"
+		(property "Footprint" "JT_USB_C:UP20-C-F-G-FL-1-P12-TR"
 			(at 26.67 69.85 0)
 			(effects

Commit message: All components placed (no traces yet tho)
Parts:
- added H403, H404, H405, H406, H407: MountingHole, MountingHole:MountingHole_2.2mm_M2, symbol Mechanical:MountingHole
Connections:
- net at R407.1: now also D405.1 (K)

Commit message: push pcb
Parts:
- C401, C402: footprint Capacitor_SMD:C_0603_1608Metric -> Capacitor_SMD:C_0805_2012Metric
Changed lines of the file:
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@@
 			)
 		)
-		(property "Footprint" "Capacitor_SMD:C_0603_1608Metric"
+		(property "Footprint" "Capacitor_SMD:C_0805_2012Metric"
 			(at 120.015 95.885 0)
 			(effects
@@
 			)
 		)
-		(property "Footprint" "Capacitor_SMD:C_0603_1608Metric"
+		(property "Footprint" "Capacitor_SMD:C_0805_2012Metric"
 			(at 127.635 95.885 0)
 			(effects
@@
 		(dnp no)
 		(property "Reference" "D403"
-			(at 191.516 95.758 0)
-			(effects
-				(font
+			(at 190.246 95.758 0)
+			(effects
+				(font

Commit message: Push non terminé
Other:
- company: (none) -> C3I
- title: (none) -> Hub USB2.0 Pomodoro
Changed lines of the file:
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@@
 	(generator_version "9.0")
 	(paper "A4")
+	(title_block
+		(title "Hub USB2.0 Pomodoro")
+		(date "2025-04-20")
+		(rev "1.0")
+		(company "C3I")
+		(comment 1 "Jacob Turcotte")
+		(comment 2 "&")
+		(comment 3 "Charles-Ariel Dion")
+		(comment 4 "Par: Équipe 3")
+	)
 	(rectangle
 		(start 64.77 17.78)
